File: Backscatter_Comms_Board/_autosave-Backscatter_Comms_Board.kicad_pcb (KiCad board)
At the start: 2 copper layers, 43 parts, among them J1 Conn_01x03, J2 Conn_01x07, J3 Conn_01x02, M1 MNMOS, M2 MNMOS, T1 SP-48, U1 ADG919BRMZ, U2 ADG841YKSZ-REEL7, U3 NCS2200SQ2T2G

Commit message: Meeting notes
Parts:
- moved J1 95.9 mm to (137.8, 89.5), turned to 270 degrees
- moved L1 72.7 mm to (135.3, 73.7), turned to 270 degrees
- moved M2 71.9 mm to (133.3, 81.3)
- moved L2 71.5 mm to (131.4, 74.3), turned to 180 degrees
- moved C1 68.5 mm to (135.3, 70.2), turned to 270 degrees
- moved C2 66.8 mm to (134.0, 76.8)
- moved U1 63.1 mm to (130.8, 71.1), turned to 0 degrees
- moved C7 60.3 mm to (138.9, 70.1)
- moved C8 60.3 mm to (138.9, 75.3)
- moved C9 60.2 mm to (138.9, 80.4)
- moved C10 60.2 mm to (138.9, 85.6)
- moved C16 59.7 mm to (146.9, 83.4)
- moved C15 59.5 mm to (146.9, 78.3)
- moved C14 59.1 mm to (146.9, 73.1)
- moved M1 58.9 mm to (133.3, 85.1), turned to 0 degrees
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Routing:
- net Net-(C10-Pad1): track 0.00 -> 18.2 mm
- net Ant: track 0.00 -> 13.9 mm
- net Vrect: track 0.00 -> 13.1 mm
- net Net-(C11-Pad1): track 0.00 -> 12.3 mm
- net Net-(C19-Pad1): track 0.00 -> 11.4 mm
- net Net-(C16-Pad2): track 0.00 -> 11.3 mm
- net Net-(C15-Pad2): track 0.00 -> 11.3 mm
- net Net-(C12-Pad2): track 0.00 -> 11.0 mm
- net Net-(C14-Pad2): track 0.74 -> 11.3 mm
- net Net-(C4-Pad1): track 0.00 -> 10.0 mm
- net Stage4: track 0.00 -> 7.86 mm
- net RF_RX: track 0.00 -> 7.19 mm
- net Net-(C2-Pad1): track 0.00 -> 6.50 mm
- net Net-(C20-Pad1): track 0.00 -> 6.41 mm
- net Net-(J1-Pad3): track 0.00 -> 6.29 mm
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