File: Backscatter_Comms_Board/_autosave-Backscatter_Comms_Board.kicad_pcb (KiCad board)
At the start: 2 copper layers, 23.5 x 24.4 mm, 75 parts, among them IC1 BQ25570, IC2 MSP430FR2100IPW16, J1 Conn_01x04, J2 SPK_IN, J4 Conn_Coaxial_Power, T2 SP-48, U2 ADG919BCPZ-REEL7, U3 SI1016X-T1-GE3, U4 TPS780270200DDCT, U5 ADG841YKSZ-REEL7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

Commit message: trying to make commit workj >:(
Routing:
- net GND: track 62.0 -> 63.7 mm
Other:
- board text removed: "Ad 0 ohm resistors to MCU connections"
- board text removed: "Add gnd Vias"
- board text removed: "Add switch option tp spk_en"
- board text removed: "Coplanar wave guide calculations"
- board text removed: "Make 4-layer"
Changed lines of the file:
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@@
   (general
     (thickness 1.6)
-    (drawings 9)
-    (tracks 342)
+    (drawings 4)
+    (tracks 346)
     (zones 0)
     (modules 75)
@@
     )
   )
-  (gr_text "Coplanar wave guide calculations\n" (at 217.2716 141.2748) (layer F.Cu)
-    (effects (font (size 1.5 1.5) (thickness 0.3)))
-  )
-  (gr_text "Add gnd Vias\n" (at 205.4098 138.6078) (layer F.Cu)
-    (effects (font (size 1.5 1.5) (thickness 0.3)))
-  )
-  (gr_text "Make 4-layer\n" (at 205.2066 135.7122) (layer F.Cu)
-    (effects (font (size 1.5 1.5) (thickness 0.3)))
-  )
   (gr_line (start 170.248516 138.670137) (end 170.106 139.573) (layer Edge.Cuts) (width 0.05))
   (gr_line (start 170.106 147.28) (end 170.106 148.0058) (layer Edge.Cuts) (width 0.05))
-  (gr_text "Ad 0 ohm resistors to MCU connections\n" (at 205.5622 113.6904) (layer F.Cu)
-    (effects (font (size 1.5 1.5) (thickness 0.3)))
-  )
-  (gr_text "Add switch option tp spk_en\n\n" (at 207.4672 128.778) (layer F.Cu)
-    (effects (font (size 1.5 1.5) (thickness 0.3)))
-  )
   (gr_line (start 170.106 143.78) (end 170.106 139.573) (layer Edge.Cuts) (width 0.05))
   (gr_arc (start 181.4464 143.51) (end 170.106 148.0058) (angle -315) (layer Edge.Cuts) (width 0.05))
@@
   (segment (start 182.9308 142.082774) (end 182.5371 142.476474) (width 0.1524) (layer F.Cu) (net 2))
   (segment (start 182.9308 141.7574) (end 182.9308 142.082774) (width 0.1524) (layer F.Cu) (net 2))
+  (segment (start 186.8849 142.9976) (end 186.9059 142.9766) (width 0.254) (layer F.Cu) (net 2))
+  (segment (start 186.8849 143.8376) (end 186.8849 142.9976) (width 0.254) (layer F.Cu) (net 2))
+  (segment (start 186.8849 144.6751) (end 186.8689 144.6911) (width 0.254) (layer F.Cu) (net 2))
+  (segment (start 186.8849 143.8376) (end 186.8849 144.6751) (width 0.254) (layer F.Cu) (net 2))
   (segment (start 178.4858 136.8392) (end 178.5032 136.8218) (width 0.1524) (layer B.Cu) (net 3))
   (segment (start 177.7862 136.8044) (end 177.8508 136.8044) (width 0.1524) (layer F.Cu) (net 3))
