File: Backscatter_Comms_Board/_autosave-Backscatter_Comms_Board.sch (KiCad schematic (older format))
At the start: 45 parts, among them J1 SPK_IN, J2 Conn_01x09, J3 Conn_01x02, M1 MNMOS, M2 DNP, T1 SP-48, U1 ADG919BRMZ, U2 ADG841YKSZ-REEL7, U3 NCS2200SQ2T2G

Commit message: Redid Board layou
Even smaller rf path and other fun things
Parts:
- added R4, R5, R6: 0, Resistor_SMD:R_0805_2012Metric, symbol Device:R_US
Connections:
- net Ant: now also R6.1; no longer C3.1, L3.1
- net at C2.1, L2.1: now also R5.2; no longer U1.5 (RF2)
- net at C1.2, L1.1: now also R4.2; no longer U1.8 (RF1)
- new net: R5.1, U1.5 (RF2)
- new net: R4.1, U1.8 (RF1)
- new net: C3.1, L3.1, R6.2
Changed lines of the file:
@@
 Wire Wire Line
 	2450 2500 3250 2500
-Connection ~ 3250 2500
 Wire Wire Line
 	6000 3150 6000 3000
@@
 	8250 2400 8250 2500
 Wire Wire Line
-	3250 2500 4250 2500
-Wire Wire Line
 	4250 2500 4250 2600
-Connection ~ 4250 2500
 Wire Wire Line
 	4250 2500 4350 2500
@@
 AN_EN
 Wire Wire Line
-	2650 4500 3500 4500
-Wire Wire Line
-	3500 5000 3000 5000
-Wire Wire Line
 	3000 5000 3000 4600
-Connection ~ 3500 4500
 Wire Wire Line
 	3000 4600 2650 4600
-Connection ~ 3500 5000
 Wire Wire Line
 	3500 4500 4100 4500
@@
 	1    0    0    -1
 $EndComp
+$Comp
+L Device:R_US R6
+U 1 1 6100CECF
+P 3750 2500
+F 0 "R6" H 3818 2546 50  0000 L CNN
+F 1 "0" H 3818 2455 50  0000 L CNN
+F 2 "Resistor_SMD:R_0805_2012Metric" V 3790 2490 50  0001 C CNN
+F 3 "~" H 3750 2500 50  0001 C CNN
+	1    3750 2500
+	0    -1   -1   0
+$EndComp
+Wire Wire Line
+	3250 2500 3600 2500
+Connection ~ 3250 2500
+Wire Wire Line
+	3900 2500 4250 2500
+Connection ~ 4250 2500
+$Comp
+L Device:R_US R5
+U 1 1 6102CCD2
+P 3250 5000
+F 0 "R5" H 3318 5046 50  0000 L CNN
+F 1 "0" H 3318 4955 50  0000 L CNN
+F 2 "Resistor_SMD:R_0805_2012Metric" V 3290 4990 50  0001 C CNN
+F 3 "~" H 3250 5000 50  0001 C CNN
+	1    3250 5000
+	0    -1   -1   0
+$EndComp
+$Comp
+L Device:R_US R4
+U 1 1 61033385
+P 3100 4500
+F 0 "R4" H 3168 4546 50  0000 L CNN
+F 1 "0" H 3168 4455 50  0000 L CNN
+F 2 "Resistor_SMD:R_0805_2012Metric" V 3140 4490 50  0001 C CNN
+F 3 "~" H 3100 4500 50  0001 C CNN
+	1    3100 4500
+	0    -1   -1   0
+$EndComp
+Wire Wire Line
+	2650 4500 2950 4500
+Wire Wire Line
+	3250 4500 3500 4500
+Connection ~ 3500 4500
+Wire Wire Line
+	3400 5000 3500 5000
+Connection ~ 3500 5000
+Wire Wire Line
+	3100 5000 3000 5000
 $EndSCHEMATC
