File: Backscatter_Comms_Board/Backscatter_Comms_Board.sch (KiCad schematic (older format))
At the start: 43 parts, among them J1 Conn_01x03, J2 Conn_01x07, J3 Conn_01x02, M1 MNMOS, M2 MNMOS, T1 SP-48, U1 ADG919BRMZ, U2 ADG841YKSZ-REEL7, U3 NCS2200SQ2T2G

Commit message: rolled back cause the PCB broke
Parts:
- added C?: 0.01uF, Capacitor_SMD:C_0805_2012Metric, symbol Device:C
- J1: value Conn_01x03 -> SPK_IN
- M2: value MNMOS -> DNP
Connections:
- net labels added: RX_EN
- wire segments 138 -> 140
Other:
- note added: "*Filter values may change\n"
- note added: "CHANGE FROM HEADER TO MIC"
- note added: "Change ant to SMA for ease of use\n"
Changed lines of the file:
@@
 P 4250 5700
 F 0 "M2" H 4537 5746 50  0000 L CNN
-F 1 "MNMOS" H 4537 5655 50  0000 L CNN
+F 1 "DNP" H 4537 5655 50  0000 L CNN
 F 2 "Local Components:BF1101WR" H 4225 5700 50  0001 C CNN
 F 3 "~" H 4225 5700 50  0001 C CNN
@@
 P 4600 6800
 F 0 "J1" V 4472 6980 50  0000 L CNN
-F 1 "Conn_01x03" V 4563 6980 50  0000 L CNN
+F 1 "SPK_IN" V 4563 6980 50  0000 L CNN
 F 2 "Connector_PinHeader_1.00mm:PinHeader_1x03_P1.00mm_Vertical" H 4600 6800 50  0001 C CNN
 F 3 "~" H 4600 6800 50  0001 C CNN
@@
 	6100 6750 5850 6750
 Wire Wire Line
-	6100 6850 5850 6850
+	6100 6950 5850 6950
 Text GLabel 5850 6550 0    50   Input ~ 0
 Stage4
 Text GLabel 5850 6750 0    50   Input ~ 0
 RF_RX
-Text GLabel 5850 6950 0    50   Input ~ 0
+Text GLabel 5850 7050 0    50   Input ~ 0
 SPK_EN
 Text GLabel 7500 4000 2    50   Input ~ 0
@@
 Wire Wire Line
 	6750 2500 7000 2500
-Text GLabel 5850 7050 0    50   Input ~ 0
+Text GLabel 5850 7150 0    50   Input ~ 0
 AN_EN
-Text GLabel 5850 7150 0    50   Input ~ 0
+Text GLabel 5850 7250 0    50   Input ~ 0
 Ant
 $Comp
@@
 $EndComp
 Wire Wire Line
-	6100 6950 5850 6950
-Wire Wire Line
-	5850 7050 6100 7050
-Wire Wire Line
-	6100 7150 5850 7150
+	6100 7050 5850 7050
+Wire Wire Line
+	5850 7150 6100 7150
+Wire Wire Line
+	6100 7250 5850 7250
 Wire Wire Line
 	9150 5050 9700 5050
@@
 $EndComp
 Connection ~ 6750 6000
-Text GLabel 5850 6850 0    50   Input ~ 0
+Text GLabel 5850 6950 0    50   Input ~ 0
 UPLINK_SR
 $Comp
@@
 	0    -1   1    0
 $EndComp
+Wire Wire Line
+	1700 4200 1700 4100
+$Comp
+L power:GND #PWR?
+U 1 1 60ED2153
+P 1700 4100
+F 0 "#PWR?" H 1700 3850 50  0001 C CNN
+F 1 "GND" H 1705 3927 50  0000 C CNN
+F 2 "" H 1700 4100 50  0001 C CNN
+F 3 "" H 1700 4100 50  0001 C CNN
+	1    1700 4100
+	-1   0    0    1
+$EndComp
+$Comp
+L Device:C C?
+U 1 1 60ED2159
+P 1700 4350
+F 0 "C?" H 1815 4396 50  0000 L CNN
+F 1 "0.01uF" H 1815 4305 50  0000 L CNN
+F 2 "Capacitor_SMD:C_0805_2012Metric" H 1738 4200 50  0001 C CNN
+F 3 "~" H 1700 4350 50  0001 C CNN
+	1    1700 4350
+	-1   0    0    1
+$EndComp
+Text GLabel 5850 6850 0    50   Input ~ 0
+RF_TX
+Wire Wire Line
+	6100 6850 5850 6850
+Text GLabel 9550 1300 0    50   Input ~ 0
+RX_EN
+Text Notes 4100 7000 0    50   ~ 0
+CHANGE FROM HEADER TO MIC
+Text Notes 3700 4200 0    50   ~ 0
+*Filter values may change\n
+Text Notes 3300 4950 0    50   ~ 0
+*Filter values may change\n
+Text Notes 3750 2250 0    50   ~ 0
+*Filter values may change\n
+Text Notes 5450 7400 0    50   ~ 0
+Change ant to SMA for ease of use\n
 $EndSCHEMATC

Commit message: Too big version
Parts:
- removed J2: Conn_01x07, Connector_PinHeader_1.00mm:PinHeader_1x07_P1.00mm_Vertical, symbol Connector_Generic:Conn_01x07
- added AE1: Antenna_Chip, Connector_Coaxial:U.FL_Molex_MCRF_73412-0110_Vertical, symbol Device:Antenna_Chip
- added J2: Conn_01x09, Connector_PinHeader_1.00mm:PinHeader_1x09_P1.00mm_Vertical, symbol Connector_Generic:Conn_01x09
- J1: footprint Connector_PinHeader_1.00mm:PinHeader_1x03_P1.00mm_Vertical -> Local Components:Multi-purpose_mic
- gave numbers to parts that had none: 1
Connections:
- wire segments 140 -> 145
Other:
- note removed: "Change ant to SMA for ease of use\n"
- moved on the sheet: C22
Changed lines of the file:
@@
 Connection ~ 2750 5000
 Wire Wire Line
-	1850 4500 1500 4500
+	1850 4500 1700 4500
 Wire Wire Line
 	1850 4700 1500 4700
@@
 F 0 "J1" V 4472 6980 50  0000 L CNN
 F 1 "SPK_IN" V 4563 6980 50  0000 L CNN
-F 2 "Connector_PinHeader_1.00mm:PinHeader_1x03_P1.00mm_Vertical" H 4600 6800 50  0001 C CNN
+F 2 "Local Components:Multi-purpose_mic" H 4600 6800 50  0001 C CNN
 F 3 "~" H 4600 6800 50  0001 C CNN
 	1    4600 6800
@@
 Text GLabel 5850 7150 0    50   Input ~ 0
 AN_EN
-Text GLabel 5850 7250 0    50   Input ~ 0
+Text GLabel 5800 7550 0    50   Input ~ 0
 Ant
 $Comp
@@
 	1    0    0    -1
 $EndComp
-$Comp
-L Connector_Generic:Conn_01x07 J2
-U 1 1 60FD2669
-P 6300 6850
-F 0 "J2" H 6380 6892 50  0000 L CNN
-F 1 "Conn_01x07" H 6380 6801 50  0000 L CNN
-F 2 "Connector_PinHeader_1.00mm:PinHeader_1x07_P1.00mm_Vertical" H 6300 6850 50  0001 C CNN
-F 3 "~" H 6300 6850 50  0001 C CNN
-	1    6300 6850
-	1    0    0    -1
-$EndComp
 Wire Wire Line
 	6100 7050 5850 7050
@@
 	5850 7150 6100 7150
 Wire Wire Line
-	6100 7250 5850 7250
+	6050 7550 5800 7550
 Wire Wire Line
 	9150 5050 9700 5050
@@
 $EndComp
 Wire Wire Line
-	1700 4200 1700 4100
-$Comp
-L power:GND #PWR?
+	1700 4100 1700 4000
+$Comp
+L power:GND #PWR0101
 U 1 1 60ED2153
-P 1700 4100
-F 0 "#PWR?" H 1700 3850 50  0001 C CNN
-F 1 "GND" H 1705 3927 50  0000 C CNN
-F 2 "" H 1700 4100 50  0001 C CNN
-F 3 "" H 1700 4100 50  0001 C CNN
-	1    1700 4100
+P 1700 4000
+F 0 "#PWR0101" H 1700 3750 50  0001 C CNN
+F 1 "GND" H 1705 3827 50  0000 C CNN
+F 2 "" H 1700 4000 50  0001 C CNN
+F 3 "" H 1700 4000 50  0001 C CNN
+	1    1700 4000
 	-1   0    0    1
 $EndComp
 $Comp
-L Device:C C?
+L Device:C C22
 U 1 1 60ED2159
-P 1700 4350
-F 0 "C?" H 1815 4396 50  0000 L CNN
-F 1 "0.01uF" H 1815 4305 50  0000 L CNN
-F 2 "Capacitor_SMD:C_0805_2012Metric" H 1738 4200 50  0001 C CNN
-F 3 "~" H 1700 4350 50  0001 C CNN
-	1    1700 4350
+P 1700 4250
+F 0 "C22" H 1815 4296 50  0000 L CNN
+F 1 "0.01uF" H 1815 4205 50  0000 L CNN
+F 2 "Capacitor_SMD:C_0805_2012Metric" H 1738 4100 50  0001 C CNN
+F 3 "~" H 1700 4250 50  0001 C CNN
+	1    1700 4250
 	-1   0    0    1
 $EndComp
@@
 Text Notes 3750 2250 0    50   ~ 0
 *Filter values may change\n
-Text Notes 5450 7400 0    50   ~ 0
-Change ant to SMA for ease of use\n
+$Comp
+L Device:Antenna_Chip AE1
+U 1 1 60EE6BC8
+P 6150 7450
+F 0 "AE1" V 6122 7754 50  0000 L CNN
+F 1 "Antenna_Chip" V 6213 7754 50  0000 L CNN
+F 2 "Connector_Coaxial:U.FL_Molex_MCRF_73412-0110_Vertical" H 6050 7625 50  0001 C CNN
+F 3 "~" H 6050 7625 50  0001 C CNN
+	1    6150 7450
+	0    1    1    0
+$EndComp
+$Comp
+L power:GND #PWR0102
+U 1 1 60EEE4F1
+P 5800 7350
+F 0 "#PWR0102" H 5800 7100 50  0001 C CNN
+F 1 "GND" H 5805 7177 50  0000 C CNN
+F 2 "" H 5800 7350 50  0001 C CNN
+F 3 "" H 5800 7350 50  0001 C CNN
+	1    5800 7350
+	0    1    1    0
+$EndComp
+Wire Wire Line
+	6050 7350 5800 7350
+Wire Wire Line
+	1700 4400 1700 4500
+Connection ~ 1700 4500
+Wire Wire Line
+	1700 4500 1500 4500
+Text GLabel 5850 6450 0    50   Input ~ 0
+RX_EN
+Text GLabel 5850 6350 0    50   Input ~ 0
+Vstore
+Wire Wire Line
+	5850 6450 6100 6450
+Wire Wire Line
+	5850 6350 6100 6350
+$Comp
+L Connector_Generic:Conn_01x09 J2
+U 1 1 60F82694
+P 6300 6750
+F 0 "J2" H 6380 6792 50  0000 L CNN
+F 1 "Conn_01x09" H 6380 6701 50  0000 L CNN
+F 2 "Connector_PinHeader_1.00mm:PinHeader_1x09_P1.00mm_Vertical" H 6300 6750 50  0001 C CNN
+F 3 "~" H 6300 6750 50  0001 C CNN
+	1    6300 6750
+	1    0    0    -1
+$EndComp
 $EndSCHEMATC

Commit message: Routed Main components
All components routed except the i/o pins
Parts:
- added R4, R5, R6: 0, Resistor_SMD:R_0402_1005Metric_Pad0.72x0.64mm_HandSolder, symbol Device:R_US
- AE1: footprint Connector_Coaxial:U.FL_Molex_MCRF_73412-0110_Vertical -> Connector_Coaxial:MMCX_Molex_73415-0961_Horizontal_1.0mm-PCB
- C1, C10, C11, C12, C13, C14, C15, C16, C17, C18, C19, C2, C20, C21, C22, C3, C4, C5, C6, C7, C8, C9: footprint Capacitor_SMD:C_0805_2012Metric -> Capacitor_SMD:C_0402_1005Metric_Pad0.74x0.62mm_HandSolder
- J2: footprint Connector_PinHeader_1.00mm:PinHeader_1x09_P1.00mm_Vertical -> Connector_PinHeader_2.54mm:PinHeader_1x09_P2.54mm_Vertical
- J3: footprint Connector_PinHeader_1.00mm:PinHeader_1x02_P1.00mm_Vertical -> Connector_PinHeader_2.54mm:PinHeader_1x02_P2.54mm_Vertical
- R1, R2, R3: footprint Resistor_SMD:R_0805_2012Metric -> Resistor_SMD:R_0402_1005Metric_Pad0.72x0.64mm_HandSolder
Connections:
- wire segments 145 -> 148
Other:
- note added: "Add downlink_SR\n"

Commit message: Final?
This will be the final of today unless we decide to do a design review
Parts:
- removed M1: MNMOS, Local Components:BF1101WR, symbol pspice:MNMOS
- removed M2: DNP, Local Components:BF1101WR, symbol pspice:MNMOS
- added DNP1: R_DLS, Resistor_SMD:R_0402_1005Metric_Pad0.72x0.64mm_HandSolder, symbol Device:R_US
- added M1, M2: BF1101WR, Local Components:BF1101WR, symbol ADG919:BF1101WR
- AE1: footprint Connector_Coaxial:MMCX_Molex_73415-0961_Horizontal_1.0mm-PCB -> Connector_Coaxial:MMCX_Molex_73415-0961_Horizontal_0.8mm-PCB
Connections:
- wire segments 148 -> 151
Changed lines of the file:
@@
 Wire Wire Line
 	4050 5500 4050 5600
-$Comp
-L pspice:MNMOS M2
-U 1 1 60EC15C1
-P 4250 5700
-F 0 "M2" H 4537 5746 50  0000 L CNN
-F 1 "DNP" H 4537 5655 50  0000 L CNN
-F 2 "Local Components:BF1101WR" H 4225 5700 50  0001 C CNN
-F 3 "~" H 4225 5700 50  0001 C CNN
-	1    4250 5700
-	0    1    -1   0
-$EndComp
 Wire Wire Line
 	4050 5500 3500 5500
 Wire Wire Line
 	3500 5500 3500 5300
-Connection ~ 4050 5500
 Wire Wire Line
 	3500 5500 3500 5750
@@
 $EndComp
 Wire Wire Line
+	6100 6350 5850 6350
+Wire Wire Line
+	6100 6950 5850 6950
+Wire Wire Line
+	6100 7150 5850 7150
+Wire Wire Line
 	6100 6550 5850 6550
-Wire Wire Line
-	6100 6650 5850 6650
-Wire Wire Line
-	6100 6750 5850 6750
-Wire Wire Line
-	6100 6950 5850 6950
-Text GLabel 5850 6550 0    50   Input ~ 0
+Text GLabel 5850 6350 0    50   Input ~ 0
 Stage4
-Text GLabel 5850 6750 0    50   Input ~ 0
+Text GLabel 5850 7150 0    50   Input ~ 0
 RF_RX
-Text GLabel 5850 7050 0    50   Input ~ 0
-SPK_EN
 Text GLabel 7500 4000 2    50   Input ~ 0
 Stage4
@@
 Wire Wire Line
 	6750 2500 7000 2500
-Text GLabel 5850 7150 0    50   Input ~ 0
+Text GLabel 5850 6850 0    50   Input ~ 0
 AN_EN
 Text GLabel 5800 7550 0    50   Input ~ 0
@@
 $EndComp
 Wire Wire Line
-	6100 7050 5850 7050
-Wire Wire Line
-	5850 7150 6100 7150
-Wire Wire Line
 	6050 7550 5800 7550
 Wire Wire Line
@@
 Wire Wire Line
 	8350 5450 8000 5450
-Wire Wire Line
-	9700 5650 9500 5650
-Wire Wire Line
-	9500 5650 9500 6000
 Text GLabel 8000 5450 0    50   Input ~ 0
 Vstore
@@
 Wire Wire Line
 	9150 5450 9150 5650
-Wire Wire Line
-	9150 5650 9500 5650
-Connection ~ 9500 5650
 Wire Wire Line
 	10300 5650 10500 5650
@@
 $EndComp
 Connection ~ 6750 6000
-Text GLabel 5850 6950 0    50   Input ~ 0
+Text GLabel 5850 6550 0    50   Input ~ 0
 UPLINK_SR
 $Comp
@@
 	1    0    0    -1
 $EndComp
-Text GLabel 5850 6650 0    50   Input ~ 0
+Text GLabel 5850 6950 0    50   Input ~ 0
 Vrect
 $Comp
@@
 	1    0    0    -1
 $EndComp
-$Comp
-L pspice:MNMOS M1
-U 1 1 60E5009C
-P 3350 3100
-F 0 "M1" H 3637 3146 50  0000 L CNN
-F 1 "MNMOS" H 3637 3055 50  0000 L CNN
-F 2 "Local Components:BF1101WR" H 3325 3100 50  0001 C CNN
-F 3 "~" H 3325 3100 50  0001 C CNN
-	1    3350 3100
-	-1   0    0    -1
-$EndComp
-Wire Wire Line
-	3250 3300 3200 3300
-Text GLabel 3550 3100 2    50   Input ~ 0
+Text GLabel 3650 3100 2    50   Input ~ 0
 RF_TX
-$Comp
-L power:GND #PWR02
-U 1 1 6106FF9F
-P 3200 3300
-F 0 "#PWR02" H 3200 3050 50  0001 C CNN
-F 1 "GND" H 3205 3127 50  0000 C CNN
-F 2 "" H 3200 3300 50  0001 C CNN
-F 3 "" H 3200 3300 50  0001 C CNN
-	1    3200 3300
-	1    0    0    -1
-$EndComp
-Connection ~ 3200 3300
-Wire Wire Line
-	3200 3300 3150 3300
 Wire Wire Line
 	3250 2500 3250 2900
@@
 	-1   0    0    1
 $EndComp
-Text GLabel 5850 6850 0    50   Input ~ 0
+Text GLabel 5850 6750 0    50   Input ~ 0
 RF_TX
-Wire Wire Line
-	6100 6850 5850 6850
 Text GLabel 9550 1300 0    50   Input ~ 0
 RX_EN
@@
 F 0 "AE1" V 6122 7754 50  0000 L CNN
 F 1 "Antenna_Chip" V 6213 7754 50  0000 L CNN
-F 2 "Connector_Coaxial:MMCX_Molex_73415-0961_Horizontal_1.0mm-PCB" H 6050 7625 50  0001 C CNN
+F 2 "Connector_Coaxial:MMCX_Molex_73415-0961_Horizontal_0.8mm-PCB" H 6050 7625 50  0001 C CNN
 F 3 "~" H 6050 7625 50  0001 C CNN
 	1    6150 7450
@@
 	1700 4500 1500 4500
 Text GLabel 5850 6450 0    50   Input ~ 0
-RX_EN
-Text GLabel 5850 6350 0    50   Input ~ 0
 Vstore
 Wire Wire Line
 	5850 6450 6100 6450
-Wire Wire Line
-	5850 6350 6100 6350
 $Comp
 L Connector_Generic:Conn_01x09 J2
@@
 Text Notes 9650 5950 0    50   ~ 0
 Add downlink_SR\n
+Wire Wire Line
+	6100 6650 5850 6650
+Text GLabel 5850 6650 0    50   Input ~ 0
+SPK_EN
+Wire Wire Line
+	5850 7050 6100 7050
+Text GLabel 5850 7050 0    50   Input ~ 0
+RX_EN
+$Comp
+L ADG919:BF1101WR M1
+U 1 1 6104D965
+P 3350 3100
+F 0 "M1" H 3538 3146 50  0000 L CNN
+F 1 "BF1101WR" H 3538 3055 50  0000 L CNN
+F 2 "Local Components:BF1101WR" H 3325 3100 50  0001 C CNN
+F 3 "~" H 3325 3100 50  0001 C CNN
+	1    3350 3100
+	-1   0    0    -1
+$EndComp
+$Comp
+L power:GND #PWR02
+U 1 1 6106FF9F
+P 3250 3300
+F 0 "#PWR02" H 3250 3050 50  0001 C CNN
+F 1 "GND" H 3255 3127 50  0000 C CNN
+F 2 "" H 3250 3300 50  0001 C CNN
+F 3 "" H 3250 3300 50  0001 C CNN
+	1    3250 3300
+	1    0    0    -1
+$EndComp
+Wire Wire Line
+	3650 3100 3550 3100
+Wire Wire Line
+	3550 3100 3550 3050
+Wire Wire Line
+	3550 3100 3550 3150
+Connection ~ 3550 3100
+$Comp
+L ADG919:BF1101WR M2
+U 1 1 6107F5AB
+P 4250 5700
+F 0 "M2" V 4575 5700 50  0000 C CNN
+F 1 "BF1101WR" V 4484 5700 50  0000 C CNN
+F 2 "Local Components:BF1101WR" H 4225 5700 50  0001 C CNN
+F 3 "~" H 4225 5700 50  0001 C CNN
+	1    4250 5700
+	0    1    -1   0
+$EndComp
+Wire Wire Line
+	4300 5900 4250 5900
+Connection ~ 4250 5900
+Wire Wire Line
+	4250 5900 4200 5900
+Wire Wire Line
+	6100 6750 5850 6750
+Wire Wire Line
+	5850 6850 6100 6850
+Wire Wire Line
+	9150 5650 9500 5650
+$Comp
+L Device:R_US DNP1
+U 1 1 6110FF1A
+P 9500 5850
+F 0 "DNP1" H 9568 5896 50  0000 L CNN
+F 1 "R_DLS" H 9568 5805 50  0000 L CNN
+F 2 "Resistor_SMD:R_0402_1005Metric_Pad0.72x0.64mm_HandSolder" V 9540 5840 50  0001 C CNN
+F 3 "~" H 9500 5850 50  0001 C CNN
+	1    9500 5850
+	-1   0    0    1
+$EndComp
+Wire Wire Line
+	9500 5700 9500 5650
+Connection ~ 9500 5650
+Wire Wire Line
+	9500 5650 9700 5650
 $EndSCHEMATC
